File: nano_IPBL_2026.kicad_pcb (KiCad board)
At the start: 2 copper layers, 44 x 85 mm, 23 parts, among them J3 DB301V-5.0-2P, M1 Motor_Servo, M10 Motor_Servo, M11 Motor_Servo, M12 Motor_Servo, M2 Motor_Servo, M3 Motor_Servo, M4 Motor_Servo, M5 Motor_Servo, M6 Motor_Servo, M7 Motor_Servo, M8 Motor_Servo, M9 Motor_Servo

Commit message: Update PCB design to revision 3.3 and schematic to revision 2.1
- Remove RX/TX mounting holes from schematic
- Prepare for servo pin net label updates
Parts:
- removed RX1, TX1: MountingHole_Pad, Arduino_MountingHole:MountingHole_1.2mm_M2_Pad_EDITED
- moved M12 5.08 mm to (112.6, 120.0), turned to 0 degrees
- moved M2 3.93 mm to (116.6, 96.8)
- moved M1 3.93 mm to (120.5, 96.8)
- moved J1 2.10 mm to (108.0, 58.4)
- renumbered J3 to J1, H1 to SW_A1, H2 to SW_B1
Connections:
- net Net-(A1-D2) renamed /D2
- A1 pad 1: Net-(A1-D1/TX) -> unconnected-(A1-D1/TX-Pad1)
- A1 pad 2: Net-(A1-D0/RX) -> unconnected-(A1-D0/RX-Pad2)
Routing:
- net Net-(A1-VIN): track 159.4 -> 203.2 mm
- net Net-(A1-D13): track 32.6 -> 44.7 mm
- net Net-(A1-D1/TX): track 5.18 -> 0.00 mm
- net Net-(A1-D0/RX): track 4.34 -> 0.00 mm
- net Net-(A1-D3): track 16.6 -> 12.7 mm
- net /D2: track 11.6 -> 8.44 mm
- net Net-(A1-D7): track 41.6 -> 39.1 mm
- net Net-(A1-D10): track 49.0 -> 46.8 mm
- net Net-(A1-D9): track 46.5 -> 44.3 mm
- net Net-(A1-D8): track 44.1 -> 42.0 mm
- net VCC: track 10.9 -> 11.6 mm
Other:
- board text added: "PCB Design Rev3.3"
- board text removed: "PCB Design v3.2"
